File: hardware/watch/epd_watch.kicad_pcb (KiCad board)
At the start: 4 copper layers, 34.5 x 39 mm, 63 parts, among them P1 FPC, Q1 Si1308EDL, Q2 AO3401A, Q3 Si1308EDL, SW1 BTN_UP, SW2 BTN_MIDDLE, SW3 BTN_DOWN, U1 nRF52832-QFxx, U2 XC6206PxxxMR, U3 TP4057, U4 DS3231MZ, U5 LM66100DCK, Y1 32Mhz, Y2 32.768khz

Commit message: fix battery protection whoopsie
Parts:
- removed CHARGER/SWD: SWD_interface, epd_watch:pogo_conn
- removed GPIO: GPIO, epd_watch:gpio_conn
- added J1: SWD_interface, epd_watch:pogo_conn, B.Cu at (145.4, 118.3)
- added J2: GPIO, epd_watch:gpio_conn, B.Cu at (162.6, 91.6)
- moved Q2 0.06 mm to (133.5, 111.7), turned to 0 degrees
Connections:
- C27 pad 2: Net-(Q2-D) -> Net-(Q2-S)
- Q2 pad 2: VBAT -> Net-(Q2-S)
- Q2 pad 3: Net-(Q2-D) -> VBAT
- U2 pad 3: Net-(Q2-D) -> Net-(Q2-S)
- U5 pad 6: Net-(Q2-D) -> Net-(Q2-S)
Routing:
- net Net-(Q2-D): track 8.76 -> 0.00 mm
- net Net-(Q2-S): track 0.00 -> 7.46 mm
- net Net-(Q2-G): track 5.72 -> 7.70 mm
