File: hardware/watch/epd_watch.kicad_sch (KiCad schematic)
At the start: 63 parts, among them J1 SWD_interface, J2 GPIO, P1 FPC, Q1 Si1308EDL, Q2 AO3401A, Q3 Si1308EDL, SW1 BTN_UP, SW2 BTN_MIDDLE, SW3 BTN_DOWN, U1 nRF52832-QFxx, U2 XC6206PxxxMR, U3 TP4057, U4 DS3231MZ, U5 LM66100DCK, Y1 32Mhz, Y2 32.768khz

Commit message: fix battery protection whoopsie
Connections:
- net VBAT: now also Q2.3 (D); no longer Q2.2 (S)
- net at C27.2, U2.3 (VI), U5.6 (VOUT): now also Q2.2 (S); no longer Q2.3 (D)
